File: _autosave-eps.kicad_pcb (KiCad board)
At the start: 4 copper layers, 90 x 96 mm, 43 parts, among them J1 Barrel_Jack, U1 LT3652EMSE

Commit message: v0.1Hydrogen
Other:
- board text added: "Hydrogen v0.1"
- board text added: "Ulog3"

Commit message: Solved errors
Parts:
- added J2: Conn_01x02_Pin, Connector_PinHeader_2.00mm:PinHeader_1x02_P2.00mm_Vertical, B.Cu at (126.0, 34.0)
- SC1, SC2, SC3, SC4, SC5, SC6: footprint Connector_PinHeader_1.00mm:PinHeader_2x01_P1.00mm_Vertical -> Connector_PinHeader_2.00mm:PinHeader_1x02_P2.00mm_Vertical
- moved J1 12.0 mm to (118.7, 106.0)
- moved SC6 7.27 mm to (162.0, 34.0), turned to -90 degrees
- moved SC5 5.50 mm to (156.0, 34.0), turned to -90 degrees
- moved D10 5.44 mm to (167.8, 34.1)
- moved D9 3.88 mm to (176.3, 34.0)
- moved SC4 3.79 mm to (149.9, 34.0), turned to -90 degrees
- moved SC1 2.56 mm to (131.6, 34.0), turned to -90 degrees
- moved SC3 2.25 mm to (143.8, 34.0), turned to -90 degrees
- moved REF** 1.72 mm to (103.0, 126.0)
- moved SC2 1.57 mm to (137.7, 34.0), turned to -90 degrees
- moved REF** 1.47 mm to (103.0, 36.0)
- moved REF** 1.39 mm to (187.0, 126.0)
- moved REF** 1.06 mm to (187.0, 36.0)
Connections:
- net VBUS renamed /BatteryCharger/load
Routing:
- net /BatteryCharger/load: track 33.6 -> 61.0 mm
- net GND: track 275.2 -> 302.3 mm
- net Net-(U1-SENSE): track 33.5 -> 46.2 mm
- net /BatteryCharger/in: track 100.4 -> 110.8 mm
- net Net-(D7-A): track 56.3 -> 61.5 mm
- net Net-(D2-A): track 6.74 -> 8.53 mm
- net Net-(D3-A): track 6.81 -> 8.12 mm
- net Net-(D1-A): track 6.99 -> 8.11 mm
- net Net-(D9-K): track 9.61 -> 10.7 mm
- net Net-(D4-A): track 7.36 -> 8.33 mm
- net Net-(D5-A): track 7.91 -> 8.54 mm
- net Net-(D10-K): track 9.72 -> 9.18 mm
Other:
- outline, holes or cut-outs redrawn
